File: hardware/CameraProbeUSB/CameraProbeUSB.kicad_sch (KiCad schematic)
At the start: 42 parts, among them J1 USB-A plug (IN), J2 USB-A socket (OUT), Q1 MMBT3904, Q2 MMBT3904, Q3 AO3401A, Q4 2N7002, SW1 Button, U1 AMS1117-3.3, U2 CH340C, U3 ESP-12F

Commit message: Add CameraProbe USB board schematic (Rev A), ERC clean
Parts:
- C4: footprint Capacitor_Tantalum_SMD:CP_EIA-3216-18_Kemet-A_Pad1.58x1.35mm_HandSolder -> Capacitor_Tantalum_SMD:CP_EIA-3216-18_Kemet-A

Commit message: Assign USB connector footprints; remove KiCad history and pycache from repo
Parts:
- F1: value 2A hold PTC -> 1.5A hold PTC
- J1: footprint (none) -> Connector_USB:USB_A_CNCTech_1001-011-01101_Horizontal
- J2: footprint (none) -> Connector_USB:USB_A_Molex_67643_Horizontal
Other:
- note added: "CameraProbe USB relay board Rev A - generated by tools/generate_kicad.py from DESIGN.md. J1 = CNC Tech 1001-011-01101, J2 = Molex 0676433910. Verify ESP-12F GPIO4/GPIO5 pin order against your module's datasheet."
- note removed: "CameraProbe USB relay board Rev A - generated by tools/generate_kicad.py from DESIGN.md. Assign J1/J2 footprints to match the USB connectors you buy. Verify ESP-12F GPIO4/GPIO5 pin order against your module's datasheet."

Commit message: Board outline and starting placement (Rev A)
Connections:
- net GND: now also J1.SH (SHIELD), J2.SH (SHIELD); no longer J1.5 (SHIELD), J2.5 (SHIELD)
